File: Black Rhino/PCB/black_rhino.kicad_pcb (KiCad board)
At the start: 2 copper layers, 271.5 x 115.9 mm, 174 parts, among them SW1 SW_Push, U1 ATmega32U4-AU, Y1 16MHz

Commit message: Improve Black Rhino-PCB
Parts:
- moved F1 2.45 mm to (246.9, 55.0)
Routing:
- net GND: track 191.0 -> 197.2 mm
- net Net-(C2-Pad2): track 16.1 -> 20.2 mm
- net VCC: track 7.92 -> 6.14 mm
- net +5V: track 170.5 -> 171.7 mm

Commit message: Improve Black Rhino-PCB
Parts:
- moved R1 0.76 mm to (157.7, 46.1)
- moved C3 0.76 mm to (140.5, 46.1)
- moved C7 0.76 mm to (140.5, 49.2)
- moved C4 0.73 mm to (157.7, 49.3)
- moved D28 0.70 mm to (280.3, 100.8)
- moved C5 0.19 mm to (157.0, 60.2)
- turned MX28 to 270 degrees
Routing:
- net GND: track 197.2 -> 225.3 mm
- net Net-(D28-Pad2): track 15.8 -> 8.68 mm
- net ROW1: track 442.5 -> 435.5 mm
- net +5V: track 171.7 -> 178.1 mm
- net COL13: track 199.8 -> 204.0 mm
- net Net-(C2-Pad2): track 20.2 -> 18.0 mm, vias 0 -> 2
- net VCC: track 6.14 -> 7.72 mm
- net Net-(R1-Pad2): track 40.9 -> 42.4 mm
- net Net-(D68-Pad2): track 6.92 -> 8.30 mm
- net LED0: track 51.2 -> 52.2 mm
- net COL6: track 97.0 -> 96.1 mm
- net ROW3: track 457.2 -> 458.0 mm
- net Net-(C3-Pad1): track 10.7 -> 9.93 mm

Commit message: Improve Black Rhino-PCB
Parts:
- moved R2 80.4 mm to (173.6, 53.0), turned to 0 degrees
- moved R3 78.1 mm to (173.6, 50.6), turned to 0 degrees
- moved F1 74.2 mm to (173.1, 47.5)
- moved USB1 71.1 mm to (182.4, 52.2), turned to 180 degrees
- moved SW1 28.1 mm to (209.6, 56.4)
Routing:
- net Net-(R2-Pad1): track 126.6 -> 32.8 mm
- net Net-(R3-Pad1): track 126.1 -> 35.0 mm
- net +5V: track 178.1 -> 95.6 mm
- net GND: track 225.3 -> 190.7 mm
- net Net-(R1-Pad2): track 42.4 -> 66.6 mm
- net Net-(D28-Pad2): track 8.68 -> 6.56 mm
- net Net-(C2-Pad2): track 18.0 -> 16.0 mm
- net Net-(R4-Pad2): track 5.03 -> 6.11 mm
- net VCC: track 7.72 -> 6.90 mm
- added copper zone on F.Cu, net +5V
Other:
- board text added: "+5V"
- board text added: "GND"

Commit message: Improve Black Rhino-PCB
Routing:
- net Net-(R3-Pad1): track 35.0 -> 29.5 mm
- net Net-(R2-Pad1): track 32.8 -> 28.9 mm
- net Net-(R1-Pad2): track 66.6 -> 69.2 mm
- net LED0: track 52.7 -> 53.7 mm
- net +5V: track 95.6 -> 94.8 mm

Commit message: Improve Black Rhino-PCB
Parts:
- added H23: MountingHole, MountingHole:MountingHole_2mm, B.Cu at (91.3, 81.8)
- moved H3 4.76 mm to (280.2, 158.8)
- moved H4 4.76 mm to (16.7, 158.8)
- moved SW1 1.59 mm to (209.6, 54.8), turned to 90 degrees
- moved H10 0.79 mm to (16.7, 58.7)
- moved H11 0.79 mm to (119.9, 58.7)
- moved H20 0.79 mm to (111.9, 58.7)
- moved H21 0.79 mm to (16.7, 66.7)
- moved H9 0.79 mm to (111.9, 66.7)
Routing:
- net GND: track 190.3 -> 196.8 mm, vias 1 -> 3
- net Net-(R1-Pad2): track 69.2 -> 75.0 mm
- net Net-(C2-Pad2): track 16.0 -> 17.0 mm
- net Net-(D68-Pad2): track 8.30 -> 7.68 mm
- added copper zone on F.Cu, net GND
Other:
- board size 271.5 x 115.9 mm -> 271.5 x 118.3 mm
