File: Cross River Gorilla/PCB/cross_river_gorilla.kicad_pcb (KiCad board)
At the start: 2 copper layers, 297.7 x 107.2 mm, 160 parts, among them SW1 SW_Push, U1 ATmega32U4-AU, Y1 16MHz

Commit message: Improve Cross River Gorilla-PCB
Parts:
- D65, D66: moved to F.Cu
- moved R2 180.1 mm to (129.9, 56.0), turned to 90 degrees
- moved USB1 171.9 mm to (130.9, 46.3)
- moved R5 165.2 mm to (122.9, 49.6), turned to 180 degrees
- moved F1 162.9 mm to (129.5, 65.2), turned to 90 degrees
- moved R3 162.1 mm to (132.0, 56.0), turned to 90 degrees
- moved R6 153.8 mm to (138.8, 49.6)
- moved C7 59.9 mm to (193.2, 134.7), turned to 90 degrees
- moved C3 49.4 mm to (173.9, 138.9), turned to 180 degrees
- moved C4 43.3 mm to (175.5, 148.3), turned to 180 degrees
- moved D66 40.8 mm to (228.6, 46.8), turned to 180 degrees
- moved C5 40.8 mm to (188.5, 148.2), turned to 270 degrees
- moved C6 38.6 mm to (174.6, 144.3), turned to 270 degrees
- moved D65 37.6 mm to (223.7, 46.8), turned to 180 degrees
- moved R1 25.0 mm to (174.1, 133.2)
- moved R4 15.0 mm to (192.5, 143.0), turned to 180 degrees
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Routing:
- net Net-(R1-Pad2): track 0.00 -> 169.9 mm, vias 0 -> 2
- net +5V: track 41.2 -> 196.3 mm, vias 0 -> 2
- net COL13: track 107.8 -> 262.7 mm, vias 0 -> 1
- net Net-(R2-Pad1): track 0.00 -> 141.4 mm, vias 0 -> 2
- net Net-(R3-Pad1): track 0.00 -> 140.4 mm, vias 0 -> 2
- net COL12: track 86.9 -> 217.3 mm, vias 0 -> 1
- net LED0: track 0.00 -> 116.8 mm, vias 0 -> 2
- net COL11: track 88.0 -> 198.0 mm, vias 0 -> 1
- net LED1: track 0.00 -> 105.4 mm, vias 0 -> 2
- net COL10: track 86.0 -> 175.6 mm, vias 0 -> 1
- net COL9: track 86.0 -> 147.1 mm, vias 0 -> 1
- net COL8: track 67.0 -> 122.4 mm, vias 0 -> 2
- net Net-(D66-Pad2): track 0.00 -> 52.0 mm, vias 0 -> 1
- net Net-(D65-Pad2): track 0.00 -> 46.9 mm, vias 0 -> 1
- net COL6: track 65.0 -> 107.9 mm, vias 0 -> 2
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Other:
- board size 297.7 x 107.2 mm -> 295.3 x 110.3 mm

Commit message: Improve Cross River Gorilla-PCB
Parts:
- moved H1 345.2 mm to (54.8, 149.2)
- moved H3 312.0 mm to (54.8, 48.4)
- moved H4 264.2 mm to (121.4, 79.4)
- moved H9 261.0 mm to (134.9, 135.7)
- moved H2 242.9 mm to (150.0, 60.3)
- moved H6 159.5 mm to (231.8, 135.7)
- moved H5 146.9 mm to (245.3, 60.3)
- moved H8 115.1 mm to (273.8, 79.4)
- moved H10 92.0 mm to (340.5, 149.2)
- moved H7 30.6 mm to (340.5, 48.4)
Routing:
- net GND: track 63.2 -> 71.8 mm, vias 19 -> 22
- net LED0: track 116.8 -> 111.2 mm
- net Net-(R2-Pad1): track 141.4 -> 136.6 mm
- net Net-(R3-Pad1): track 140.4 -> 136.6 mm
- net +5V: track 196.3 -> 198.2 mm
- net COL6: track 107.9 -> 108.8 mm
Other:
- board text added: "Cross River Gorilla"
